Commit message: update

File: urdf/hhfc/urdf/hhfc.urdf (robot description, URDF)
Before this commit: robot hhfc_sf, 15 links, 14 joints
Links:
- link Larm_shoulder_p: geometry visual mesh filename=package://ovinf_ros2/urdf/hhfc/meshes/Larm_shoulder_p.STL
- link Lleg_ankle_p: geometry visual mesh filename=package://ovinf_ros2/urdf/hhfc/meshes/Lleg_ankle_p.STL
- link Lleg_ankle_r: geometry collision mesh filename=package://ovinf_ros2/urdf/hhfc/meshes/whole_foot.stl; visual mesh filename=package://ovinf_ros2/urdf/hhfc/meshes/whole_foot_visual.stl
- link Lleg_hip_p: geometry visual mesh filename=package://ovinf_ros2/urdf/hhfc/meshes/Lleg_hip_p.STL
- link Lleg_hip_r: geometry visual mesh filename=package://ovinf_ros2/urdf/hhfc/meshes/Lleg_hip_r.STL
- link Lleg_hip_y: geometry visual mesh filename=package://ovinf_ros2/urdf/hhfc/meshes/Lleg_hip_y.STL
- link Lleg_knee: geometry visual mesh filename=package://ovinf_ros2/urdf/hhfc/meshes/Lleg_knee.STL
- link Rarm_shoulder_p: geometry visual mesh filename=package://ovinf_ros2/urdf/hhfc/meshes/Rarm_shoulder_p.STL
- link Rleg_ankle_p: geometry visual mesh filename=package://ovinf_ros2/urdf/hhfc/meshes/Rleg_ankle_p.STL
- link Rleg_ankle_r: geometry collision mesh filename=package://ovinf_ros2/urdf/hhfc/meshes/whole_foot.stl; visual mesh filename=package://ovinf_ros2/urdf/hhfc/meshes/whole_foot_visual.stl
- link Rleg_hip_p: geometry visual mesh filename=package://ovinf_ros2/urdf/hhfc/meshes/Rleg_hip_p.STL
- link Rleg_hip_r: geometry visual mesh filename=package://ovinf_ros2/urdf/hhfc/meshes/Rleg_hip_r.STL
- link Rleg_hip_y: geometry visual mesh filename=package://ovinf_ros2/urdf/hhfc/meshes/Rleg_hip_y.STL
- link Rleg_knee: geometry visual mesh filename=package://ovinf_ros2/urdf/hhfc/meshes/Rleg_knee.STL
- link base_thorax: geometry collision box size=0.4 0.35 0.6; visual mesh filename=package://ovinf_ros2/urdf/hhfc/meshes/base_thorax.STL
